Commit message: Modified laser_joint into laser

File: turtlebot_description/urdf/sensors/hokuyo.urdf.xacro (robot description, xacro)
@@ -4,5 +4,5 @@
 	<xacro:include filename="$(find turtlebot_description)/urdf/turtlebot_properties.urdf.xacro"/>
 	<xacro:macro name="sensor_hokuyo" params="parent">
-	<link name="laser_joint">
+	<link name="laser">
 		<collision>
 			<origin xyz="0 0 0" rpy="0 0 0"/>
@@ -27,5 +27,5 @@
 		<origin xyz="-0.145 0 0.05" rpy="0 0 1.570796"/>
 		<parent link="${parent}"/>
-		<child link="laser_joint"/>
+		<child link="laser"/>
 	</joint>
 	</xacro:macro>

Commit message: modified gazebo launch file

File: turtlebot_description/urdf/sensors/hokuyo.urdf.xacro (robot description, xacro)
@@ -25,8 +25,44 @@
 	<joint name="hokuyo_joint" type="fixed">
 		<axis xyz="0 0 1" />
-		<origin xyz="-0.145 0 0.05" rpy="0 0 1.570796"/>
+		<origin xyz="-0.125 0 0.04" rpy="0 0 1.570796"/>
 		<parent link="${parent}"/>
 		<child link="laser"/>
 	</joint>
+	  <!-- hokuyo -->
+	  <gazebo reference="sensor_hokuyo">
+		<sensor type="gpu_ray" name="head_hokuyo_sensor">
+		  <pose>0 0 0 0 0 0</pose>
+		  <visualize>true</visualize>
+		  <update_rate>40</update_rate>
+		  <ray>
+			<scan>
+			  <horizontal>
+				<samples>720</samples>
+				<resolution>1</resolution>
+				<min_angle>-1.570796</min_angle>
+				<max_angle>1.570796</max_angle>
+			  </horizontal>
+			</scan>
+			<range>
+			  <min>0.10</min>
+			  <max>30.0</max>
+			  <resolution>0.01</resolution>
+			</range>
+			<noise>
+			  <type>gaussian</type>
+			  <!-- Noise parameters based on published spec for Hokuyo laser
+				   achieving "+-30mm" accuracy at range < 10m.  A mean of 0.0m and
+				   stddev of 0.01m will put 99.7% of samples within 0.03m of the true
+				   reading. -->
+			  <mean>0.0</mean>
+			  <stddev>0.00</stddev>
+			</noise>
+		  </ray>
+		  <plugin name="gazebo_ros_head_hokuyo_controller" filename="libgazebo_ros_gpu_laser.so">
+			<topicName>/scan</topicName>
+			<frameName>laser</frameName>
+		  </plugin>
+		</sensor>
+	  </gazebo>
 	</xacro:macro>
 </robot>
